File: C-Duino/micro_new.kicad_pcb (KiCad board)
At the start: 2 copper layers, 68.6 x 53.3 mm, 47 parts, among them J1 Conn_01x08_Female, J2 Conn_01x10_Female, J3 USB_C_Receptacle_USB2.0, J4 Conn_01x08_Female, J5 Conn_01x06_Female, Q1 Q_PMOS_DGS, U1 LMV358, U2 ATMEGA32U4-AU, U3 NCP1117-5.0_SOT223, U4 LP2985-33DBVR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

Commit message: Add files via upload
Parts:
- renumbered D2 to L, D5 to LED, D1 to ON, D3 to RX, D4 to TX
